File: Hardware/StappenMotorSturing.brd (EAGLE design)
At the start: 83 x 68 mm, 79 parts, among them IC1 LPC11U24FBD48/401, Q1 PSMN0R9-25LYC, Q10 PSMN0R9-25LYC, Q2 PSMN0R9-25LYC, Q3 PSMN0R9-25LYC, Q4 PSMN0R9-25LYC, Q5 PSMN0R9-25LYC, Q6 PSMN0R9-25LYC, Q7 PSMN0R9-25LYC, Q8 PSMN0R9-25LYC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

Commit message: Added UART header, routed with airwire
Parts:
- added JP1: (no value), microbuilder:1X03_OVAL
Connections:
- new net RX: IC1.37, JP1.2
- new net TX: IC1.36, JP1.1
- net GND: now also JP1.3
Other:
- board text added: "Dit is er handmatig op gelijmd"
Changed lines of the file:
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@@
 <text x="0" y="78.74" size="1.778" layer="51">Improvement: Do not run FET Gate traces parallel to current Vin cunductor</text>
 <text x="0" y="83.82" size="1.778" layer="51">Feature: Dual connector for Phoenix MSTB and cheap chinese screw terminal</text>
+<text x="78.74" y="40.64" size="1.778" layer="51">Dit is er handmatig op gelijmd</text>
 </plain>
 <attributes>
@@
 <element name="H7" library="holes" package="3,2" value="MOUNT-HOLE3.2" x="78" y="63"/>
 <element name="H8" library="holes" package="3,2" value="MOUNT-HOLE3.2" x="5" y="63"/>
+<element name="JP1" library="microbuilder" package="1X03_OVAL" value="" x="76.2" y="43.18" rot="R90"/>
 </elements>
 <signals>
@@
 <wire x1="5.455" y1="14.002" x2="5.1" y2="14.002" width="1.016" layer="1"/>
 <wire x1="5.1" y1="14.002" x2="5.1" y2="14" width="1.016" layer="1"/>
+<contactref element="JP1" pad="3"/>
+<wire x1="76.2" y1="45.72" x2="77.47" y2="43.18" width="0" layer="19" extent="1-1"/>
 </signal>
 <signal name="N$8">
@@
 <via x="33.782" y="2.54" extent="1-16" drill="0.3302"/>
 </signal>
+<signal name="TX">
+<contactref element="IC1" pad="36"/>
+<contactref element="JP1" pad="1"/>
+<wire x1="47.482" y1="55.987" x2="76.2" y2="40.64" width="0" layer="19" extent="1-1"/>
+</signal>
+<signal name="RX">
+<contactref element="IC1" pad="37"/>
+<contactref element="JP1" pad="2"/>
+<wire x1="45.867" y1="54.372" x2="76.2" y2="43.18" width="0" layer="19" extent="1-1"/>
+</signal>
 </signals>
