File: Hardware/StappenMotorSturing.sch (EAGLE design)
At the start: 79 parts, among them IC1 LPC11U24FBD48/401, Q1 PSMN0R9-25LYC, Q10 PSMN0R9-25LYC, Q2 PSMN0R9-25LYC, Q3 PSMN0R9-25LYC, Q4 PSMN0R9-25LYC, Q5 PSMN0R9-25LYC, Q6 PSMN0R9-25LYC, Q7 PSMN0R9-25LYC, Q8 PSMN0R9-25LYC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

Commit message: Added UART header, routed with airwire
Parts:
- added JP1: (no value), microbuilder:HEADER-1X3
Connections:
- new net RX: IC1.P1.14/!DSR!/CT16B0_MAT1/RXD, JP1.2
- new net TX: IC1.P1.13/!DTR!/CT16B0_MAT0/TXD, JP1.1
- net GND: now also JP1.3
Other:
- note added: "Dit is er handmatig op gelijmd en gesoldeerd"
Changed lines of the file:
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@@
 <part name="H7" library="holes" deviceset="MOUNT-HOLE" device="3.2"/>
 <part name="H8" library="holes" deviceset="MOUNT-HOLE" device="3.2"/>
+<part name="JP1" library="microbuilder" deviceset="HEADER-1X3" device=""/>
+<part name="GND11" library="supply" deviceset="GND" device=""/>
 </parts>
 <sheets>
@@
 <wire x1="73.152" y1="55.88" x2="73.66" y2="53.34" width="0.2032" layer="97"/>
 <text x="20.32" y="226.06" size="1.9304" layer="97">Improvement: Pull down termination on HI_FET gate signals</text>
+<text x="381" y="220.98" size="1.778" layer="91">Dit is er handmatig op gelijmd en gesoldeerd</text>
 </plain>
 <instances>
@@
 <instance part="H7" gate="G$1" x="238.76" y="22.86"/>
 <instance part="H8" gate="G$1" x="264.16" y="22.86"/>
+<instance part="JP1" gate="A" x="381" y="215.9"/>
+<instance part="GND11" gate="1" x="375.92" y="205.74"/>
 </instances>
 <busses>
@@
 <pinref part="GND10" gate="1" pin="GND"/>
 <junction x="254" y="215.9"/>
+</segment>
+<segment>
+<pinref part="JP1" gate="A" pin="3"/>
+<wire x1="378.46" y1="213.36" x2="375.92" y2="213.36" width="0.2032" layer="91"/>
+<wire x1="375.92" y1="213.36" x2="375.92" y2="208.28" width="0.2032" layer="91"/>
+<pinref part="GND11" gate="1" pin="GND"/>
 </segment>
 </net>
@@
 </segment>
 </net>
+<net name="TX" class="0">
+<segment>
+<pinref part="IC1" gate="G$1" pin="P1.13/!DTR!/CT16B0_MAT0/TXD"/>
+<pinref part="JP1" gate="A" pin="1"/>
+<wire x1="370.84" y1="218.44" x2="378.46" y2="218.44" width="0.2032" layer="91"/>
+<label x="373.38" y="218.44" size="1.778" layer="95" rot="R90"/>
+</segment>
+</net>
+<net name="RX" class="0">
+<segment>
+<pinref part="IC1" gate="G$1" pin="P1.14/!DSR!/CT16B0_MAT1/RXD"/>
+<pinref part="JP1" gate="A" pin="2"/>
+<wire x1="378.46" y1="215.9" x2="370.84" y2="215.9" width="0.2032" layer="91"/>
+<label x="373.38" y="210.82" size="1.778" layer="95" rot="R90"/>
+</segment>
+</net>
